Commit message: Noetic distro update

File: robot_description/urdf/box.xacro (robot description, xacro)
@@ -1,2 +1,3 @@
+<?xml version="1.0"?>
 <robot name="box" xmlns:xacro="http://ros.org/wiki/xacro">
  <xacro:macro name="default_inertial" params="mass">
@@ -9,20 +10,20 @@
 <link name="box">
 	<visual>
-	<geometry>
-		<box size="1 1 1"/>
-	</geometry>
-	<origin xyz= "0 0 0"/>
+	   <geometry>
+		     <box size="1 1 1"/>
+     </geometry>
+	   <origin xyz= "5 0 0.5"/>
 	</visual>
 	<collision>
 		<geometry>
-		<box size="1 1 1"/>
+		    <box size="1 1 1"/>
 		</geometry>
-	<origin xyz= "0 0 0"/>
+	  <origin xyz= "5 0 0.5"/>
 	</collision>
 	<inertial>
 		<mass value="1.0"/>
 		<inertia ixx="0.17" ixy="0.0" ixz="0.0" iyy="0.17" iyz="0.0" izz="0.17" />
-		<origin xyz= "0 0 0"/>
-        </inertial>
+		<origin xyz= "5 0 0.5"/>
+  </inertial>
 </link>
 <joint name="basetoworld" type="planar">
